Commit message: new file:   build_common.sh

File: src/ugv_main/ugv_description/urdf/rasp_rover.urdf (robot description, URDF)
Before this commit: robot rasp_rover, 12 links, 11 joints
Joints:
- joint pt_camera_link_joint: origin xyz=0.047686 -0.000569 0.02 rpy=-1.5708 0 0 -> xyz=0.047686 -0.000569 0.02 rpy=3.14 -1.5708 0

File: src/ugv_main/ugv_description/urdf/ugv_beast.urdf (robot description, URDF)
Before this commit: robot ugv_beast, 13 links, 12 joints
Joints:
- joint pt_link2_to_pt_camera_link: origin xyz=0.0476858338436577 -0.000568997109077291 0.0199999999999997 rpy=-1.5707963267949 0 0 -> xyz=0.0476858338436577 -0.000568997109077291 0.0199999999999997 rpy=3.14 -1.5708 0

File: src/ugv_main/ugv_description/urdf/ugv_rover.urdf (robot description, URDF)
Before this commit: robot ugv_rover, 13 links, 12 joints
Joints:
- joint pt_link2_to_pt_camera_link: origin xyz=0.047686 -0.000569 0.02 rpy=-1.5708 0 0 -> xyz=0.047686 -0.000569 0.02 rpy=3.14 -1.5708 0

File: src/ugv_main/ugv_gazebo/urdf/rasp_rover.urdf (robot description, URDF)
Before this commit: robot rasp_rover, 12 links, 11 joints
Joints:
- joint base_lidar_link_joint: origin xyz=0.0316958390518911 -0.00101477740749894 0.0976480280297308 rpy=0 0 1.5708 -> xyz=0.0316958390518911 -0.00101477740749894 0.0976480280297308 rpy=0 0 0
- joint pt_camera_link_joint: origin xyz=0.047686 -0.000569 0.02 rpy=-1.5708 0 0 -> xyz=0.047686 -0.000569 0.02 rpy=3.14 -1.5708 0
